File: Hardware/Volt-Picker.kicad_pcb (KiCad board)
At the start: 2 copper layers, 40 x 30 mm, 61 parts, among them J1 USB_C_Receptacle, J2 Conn_01x02_Pin, Q1 SQS840CENW, Q2 MMBT2222A, Q5 SQS840CENW, U1 AP33771CFBZ-13-FA01

Commit message: ...
Parts:
- D1, D2, D3, D4: footprint tinker:PGB1010603NRHF -> LCSCfootprints:PGB1010603NRHF
- J1: footprint tinker:USB_C_Receptacle_HRO_TYPE-C-31-M-12 -> TINKERfootprints:USB_C_Receptacle_HRO_TYPE-C-31-M-12
- J2: footprint tinker:TerminalBlock_DG350-3.5-02P-14-00A(H) -> TINKERfootprints:TerminalBlock_DG350-3.5-02P-14-00A(H)
- REF**: footprint tinker:DagNabbit -> TINKERfootprints:DagNabbit
Connections:
- net FAULT renamed STATUS
Changed lines of the file:
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@@
 	(net 16 "/s-s")
 	(net 17 "Net-(LED2-K)")
-	(net 18 "FAULT")
+	(net 18 "STATUS")
 	(net 19 "Vcc")
 	(net 20 "Net-(JP1-B)")
@@
 			(size 0.725 0.2)
 			(layers "F.Cu" "F.Mask" "F.Paste")
-			(net 18 "FAULT")
+			(net 18 "STATUS")
 			(pinfunction "LED")
 			(pintype "unspecified")
@@
 		)
 	)
-	(footprint "tinker:PGB1010603NRHF"
+	(footprint "LCSCfootprints:PGB1010603NRHF"
 		(layer "F.Cu")
 		(at 107.2 103.5 -90)
@@
 		(embedded_fonts no)
 	)
-	(footprint "tinker:PGB1010603NRHF"
+	(footprint "LCSCfootprints:PGB1010603NRHF"
 		(layer "F.Cu")
 		(at 107.2 96.5 90)
@@
 		(tags "TVS Diode (Bi-directional)")
 		(property "Reference" "D4"
-			(at 2.5 0 90)
+			(at 2.5 0 270)
 			(layer "F.SilkS")
 			(effects
@@
 		)
 		(property "Value" "PGB1010603NR"
-			(at -0.415 0 90)
+			(at -0.415 0 270)
 			(layer "F.SilkS")
 			(hide yes)
@@
 		)
 		(property "Datasheet" ""
-			(at 0 0 90)
+			(at 0 0 270)
 			(layer "F.Fab")
 			(hide yes)
@@
 		)
 		(property "Description" ""
-			(at 0 0 90)
+			(at 0 0 270)
 			(layer "F.Fab")
 			(hide yes)
@@
 		)
 	)
-	(footprint "tinker:TerminalBlock_DG350-3.5-02P-14-00A(H)"
+	(footprint "TINKERfootprints:TerminalBlock_DG350-3.5-02P-14-00A(H)"
 		(layer "F.Cu")
 		(at 84.5 98.25 -90)
@@
 		)
 	)
-	(footprint "tinker:USB_C_Receptacle_HRO_TYPE-C-31-M-12"
+	(footprint "TINKERfootprints:USB_C_Receptacle_HRO_TYPE-C-31-M-12"
 		(layer "F.Cu")
 		(at 116.2 100 90)
@@
 			(layers "F.Cu" "F.Mask" "F.Paste")
 			(roundrect_rratio 0.25)
-			(net 18 "FAULT")
+			(net 18 "STATUS")
 			(pinfunction "A")
 			(pintype "passive")
@@
 		)
 	)
-	(footprint "tinker:PGB1010603NRHF"
+	(footprint "LCSCfootprints:PGB1010603NRHF"
 		(layer "F.Cu")
 		(at 105.7 96.5 90)
@@
 		(tags "TVS Diode (Bi-directional)")
 		(property "Reference" "D2"
-			(at 2.5 0 90)
+			(at 2.5 0 270)
 			(layer "F.SilkS")
 			(effects
@@
 		)
 		(property "Value" "PGB1010603NR"
-			(at -0.415 0 90)
+			(at -0.415 0 270)
 			(layer "F.SilkS")
 			(hide yes)
@@
 		)
 		(property "Datasheet" ""
-			(at 0 0 90)
+			(at 0 0 270)
 			(layer "F.Fab")
 			(hide yes)
@@
 		)
 		(property "Description" ""
-			(at 0 0 90)
+			(at 0 0 270)
 			(layer "F.Fab")
 			(hide yes)
@@
 		(embedded_fonts no)
 	)
-	(footprint "tinker:PGB1010603NRHF"
+	(footprint "LCSCfootprints:PGB1010603NRHF"
 		(layer "F.Cu")
 		(at 105.7 103.5 -90)
@@
 		(embedded_fonts no)
 	)
-	(footprint "tinker:DagNabbit"
+	(footprint "TINKERfootprints:DagNabbit"
 		(layer "B.Cu")
 		(at 111.5 100.5 -90)

Commit message: Tweakin' & Squishin'
Parts:
- moved R5 2.01 mm to (98.4, 101.0), turned to -90 degrees
- moved C3 1.19 mm to (98.5, 104.5)
- moved Q1 0.30 mm to (93.4, 97.0)
- moved JP12 0.16 mm to (105.5, 87.6)
- moved JP13 0.16 mm to (106.9, 87.6)
- moved JP14 0.16 mm to (108.4, 87.6)
- moved JP15 0.16 mm to (109.9, 87.6)
- moved JP16 0.16 mm to (111.3, 87.6)
- moved JP4 0.16 mm to (101.1, 87.6)
- moved JP5 0.16 mm to (102.6, 87.6)
- moved JP6 0.16 mm to (104.0, 87.6)
- moved R10 0.16 mm to (101.1, 89.8)
- moved R11 0.16 mm to (102.6, 89.8)
- moved R12 0.16 mm to (104.0, 89.8)
- moved R13 0.16 mm to (105.5, 89.8)
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- renumbered R8 to R2, R6 to R3, R7 to R4, R9 to R5, R5 to R6, R2 to R7
Connections:
- LED1 pad 1: Net-(LED1-K) -> GND
- LED1 pad 2: PWR_ON -> Net-(LED1-A)
- LED2 pad 1: Net-(LED2-K) -> GND
- LED2 pad 2: STATUS -> Net-(LED2-A)
- R1 pad 1: Net-(LED2-K) -> STATUS
- R1 pad 2: GND -> Net-(LED2-A)
- R2 pad 1: Net-(LED1-K) -> PWR_ON
- R2 pad 2: GND -> Net-(LED1-A)
Routing:
- net STATUS: track 12.3 -> 7.84 mm, vias 0 -> 2
- net PWR_ON: track 18.0 -> 14.6 mm, vias 2 -> 3
- net Net-(LED2-K): track 2.67 -> 0.00 mm
- net Net-(LED2-A): track 0.00 -> 2.67 mm
- net Net-(LED1-K): track 2.67 -> 0.00 mm
- net Net-(LED1-A): track 0.00 -> 2.67 mm
- net VSEL: track 31.1 -> 29.7 mm
- net Net-(U1-V5V): track 2.33 -> 1.14 mm

Commit message: One day... I'll stop tweakin'
Parts:
- F1: value 1A -> Fuse; footprint Fuse:Fuse_1206_3216Metric_Pad1.42x1.75mm_HandSolder -> Fuse:Fuseholder_Littelfuse_Nano2_154x
- J2: value Conn_01x02_Pin -> Output
- moved G*** 16.4 mm to (107.7, 110.9)
- moved JP1 12.6 mm to (88.5, 112.4)
- moved JP2 12.6 mm to (90.0, 112.4)
- moved JP3 12.6 mm to (91.5, 112.4)
- moved JP7 12.6 mm to (92.9, 112.4)
- moved JP8 12.6 mm to (94.4, 112.4)
- moved JP9 12.6 mm to (95.9, 112.4)
- moved R20 12.6 mm to (88.5, 110.2)
- moved R22 12.6 mm to (91.5, 110.2)
- moved R27 12.6 mm to (98.8, 110.2)
- moved JP10 12.6 mm to (97.3, 112.4)
- moved JP11 12.6 mm to (98.8, 112.4)
- moved R21 12.6 mm to (90.0, 110.2)
- moved R23 12.6 mm to (92.9, 110.2)
- moved R24 12.6 mm to (94.4, 110.2)
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Connections:
- F1 pad 1: Vbus -> VBUS-f
- F1 pad 2: VBUS-f -> Vbus
Routing:
- net Vbus: track 19.3 -> 18.0 mm
- net GND: vias 17 -> 16
Other:
- board text added: "${COMPANY} ${ISSUE_DATE}"
- board text added: "${TITLE} rev. ${REVISION}"
- board text removed: "${COMPANY} 2026"
- board text removed: "5V 9V 12V 15V 20V 28V rsvd rsvd"
- board text removed: "USB-PD Volt-Picker Deee-LUXE rev. ${REVISION}"
- board text removed: "auto 1A 1.5A 2A 2.5A 3A 4A 5A"
